File: electrical/ebox/ebox.sch (EAGLE design)
At the start: 48 parts, among them IC1 MAX3221CUE, IC2 MCP170350MB, IC3 XMEGA128A1, Q1 FDD4141TO252, X1 22-23-2031, X2 22-23-2031, X3 C-GRID-07-70543, X4 22-23-2021, X5 C-GRID-07-70543, X6 C-GRID-07-70543, X7 C-GRID-07-70543, X8 C-GRID-07-70543, X9 C-GRID-07-70543

Commit message: Added some packages and stuff to board.
Parts:
- added IC4: LT1161, crw:LT1161
- added X10, X11: 22-23-2041, con-molex:22-23-2041
- added X12: 22-23-2021, con-molex:22-23-2021
- added X13, X14: 22-23-2031, con-molex:22-23-2031
- U1: value BLUETOOTH-RN41" -> BLUETOOTH-RN42
- X4: value 22-23-2021 -> 22-23-2031; device con-molex:22-23-2021 -> con-molex:22-23-2031
- X8, X9: value C-GRID-07-70543 -> 22-23-2031; device con-molex:C-GRID-07-70543 -> con-molex:22-23-2031
- renumbered U$1 to U1
Connections:
- net S5_12V renamed MOT1_SIG
- removed net S5_5V: X8-4.S
- removed net S5_AN_A: X8-5.S
- removed net S5_AN_B: X8-6.S
- removed net S5_RX: X8-2.S
- removed net S5_TX: X8-3.S
- new net BATT+: X10-1.S, X11-1.S
- new net BATT-: X10-4.S, X11-4.S
- new net BATT1: X10-3.S, X11-3.S
- new net BATT2: X10-2.S, X11-2.S
- new net MOT2_SIG: X9-1.S
- net CHARGE: now also X12-1.S, X13-1.S; no longer X4-1.S
- net GND: now also X12-2.S, X13-2.S, X8-3.S, X9-3.S; no longer X4-2.S, X8-7.S
- net MOT1_A: now also X4-1.S
- net MOT1_B: now also X4-2.S
- net MOT1_C: now also X4-3.S
- net MOT2_A: now also X14-1.S
- net MOT2_B: now also X14-2.S
- net MOT2_C: now also X14-3.S
Other:
- note added: "TODO: Replace with JST"
- note added: "TODO: Replace with bullet"
- moved on the sheet: X3-1, X3-2, X3-3, X3-4, X3-5, X3-6, X3-7, X4-1, X4-2, X5-1, X5-2, X5-3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

Commit message: Added mostly complete schematic for ebox.
Parts:
- added C15: 50uF, rcl:C-USC0805
- added C16, C17, C18, C19, C20, C23, C24, C25, C26, C27, C30, C31, C32, C33, C34, C37: 0.1uF, rcl:C-USC0805
- added C21, C22, C28, C29, C35, C36, C42: 1uF, rcl:C-USC0805
- added C38: 68uF, rcl:C-USC0805
- added C39: 120uF, rcl:C-USC0805
- added C40, C41: 10uF, rcl:C-USC0805
- added D10, D5, D9: MBRA340T3, diode:MBRA340T3
- added D3, D7: (no value), zetex:D_2CSOT23
- added D4, D6, D8: GSOT05C, zetex:D_2CSOT23
- added IC10, IC13, IC14, IC17, IC18, IC5, IC6, IC9: SN74LVC1G125, crw:SN74LVC1G125
- added IC11, IC15, IC7: MAX3221CUE, maxim:MAX3221CUE
- added IC12, IC16, IC8: MCP170350MB, linear:MCP170350MB
- added IC19: 74ALS04D, 74xx-us:74ALS04D
- added IC20: AP1509-33, crw:AP1509
- added IC21, IC22: (no value), crw:INA170
- added IC23: LT3652, crw:LT3652
- added L4: 47uH, rcl:L-USL2012C
- added L5: 5.6uH, rcl:L-USL2012C
- added PTC3, PTC4, PTC5, PTC6, PTC7, PTC8: 50mA, rcl:R-US_R1206
- added R10, R11, R8, R9: 0.010, rcl:R-US_R6332
- added R12, R13, R14, R15: 2K, rcl:R-US_R0805
- added R16, R17, R18, R19: 100k, rcl:R-US_R0805
- added R20, R21: 0.05, rcl:R-US_R6332
- added R22: 626k, rcl:R-US_R0805
- added R23: 0R, rcl:R-US_R0805
- added R24: 412k, rcl:R-US_R0805
- added T2, T3, T4, T5: (no value), zetex:NMOSSOT223
Connections:
- removed net S2_AN_A: X5-5.S
- removed net S2_AN_B: X5-6.S
- removed net S3_AN_A: X6-5.S
- removed net S3_AN_B: X6-6.S
- removed net S4_AN_A: X7-5.S
- removed net S4_AN_B: X7-6.S
- new net !CHRG: IC23.!CHRG, IC3.PJ3
- new net !CHRG_FAULT: IC23.!FAULT, IC3.PJ2
- new net !EN232_1: IC19A.I, IC1G$1.!EN, IC3.PJ4
- new net !EN232_2: IC19B.I, IC3.PJ5, IC7G$1.!EN
- new net !EN232_3: IC11G$1.!EN, IC19C.I, IC3.PJ6
- new net !EN232_4: IC15G$1.!EN, IC19D.I, IC3.PJ7
- new net BATT_TEMP: IC23.NTC
- new net EN232_1: IC19A.O, IC1G$1.!FORCEOFF, IC5.!OE, IC6.!OE
- new net EN232_2: IC10.!OE, IC19B.O, IC7G$1.!FORCEOFF, IC9.!OE
- new net EN232_3: IC11G$1.!FORCEOFF, IC13.!OE, IC14.!OE, IC19C.O
- new net EN232_4: IC15G$1.!FORCEOFF, IC17.!OE, IC18.!OE, IC19D.O
- new net FAULT1: IC3.PK0, IC4.T1, R12.2
- new net FAULT2: IC3.PK2, IC4.T2, R13.2
- new net FAULT3: IC3.PK4, IC4.T3, R14.2
- new net FAULT4: IC3.PK6, IC4.T4, R15.2
- new net N$12: R8.1, T2.D
- new net N$14: R9.1, T3.D
- new net N$15: R10.1, T4.D
- new net N$16: R11.1, T5.D
- new net N$17: IC4.G1, T2.G
- new net N$18: IC4.G2, T3.G
- new net N$19: IC4.G3, T4.G
- new net N$20: IC4.G4, T5.G
- new net N$21: C16.2, IC7G$1.C1-
- new net N$22: C16.1, IC7G$1.C1+
- new net N$23: C17.2, IC7G$1.C2-
- new net N$24: C17.1, IC7G$1.C2+
- new net N$25: C18.1, IC7G$1.V+
- new net N$26: C19.2, IC7G$1.V-
- new net N$27: C23.2, IC11G$1.C1-
- new net N$28: C23.1, IC11G$1.C1+
- new net N$29: C24.2, IC11G$1.C2-
- new net N$30: C24.1, IC11G$1.C2+
- new net N$31: C25.1, IC11G$1.V+
- new net N$32: C26.2, IC11G$1.V-
- new net N$33: C30.2, IC15G$1.C1-
- new net N$34: C30.1, IC15G$1.C1+
- new net N$35: C31.2, IC15G$1.C2-
- new net N$36: C31.1, IC15G$1.C2+
- new net N$37: C32.1, IC15G$1.V+
- new net N$38: C33.2, IC15G$1.V-
- new net N$39: C41.1, IC23.TIMER
- new net N$40: D5.C, IC20.OUT, L4.1
- new net N$41: C42.2, D9.C, IC23.BOOST
- new net N$42: C42.1, D10.C, IC23.SW, L5.1
- new net N$43: D9.A, IC23.SENSE, L5.2, R20.1
- new net N$44: IC23.VFB, R23.2
- new net N$45: R22.1, R23.1, R24.2
- new net PWR_CTL1: IC3.PK1, IC4.IN1, R12.1
- new net PWR_CTL2: IC3.PK3, IC4.IN2, R13.1
- new net PWR_CTL3: IC3.PK5, IC4.IN3, R14.1
- new net PWR_CTL4: IC3.PK7, IC4.IN4, R15.1
- new net S1_RX_33V: D3.C2, IC6.A, R16.1
- new net S2_GPIO_A: PTC3.2, X5-5.S
- new net S2_GPIO_B: PTC4.2, X5-6.S
- new net S2_RX_33V: D3.C1, IC10.A, R17.1
- new net S3_GPIO_A: PTC5.2, X6-5.S
- new net S3_GPIO_B: PTC6.2, X6-6.S
- new net S3_RX_33V: D7.C2, IC14.A, R18.1
- new net S4_GPIO_A: PTC7.2, X7-5.S
- new net S4_GPIO_B: PTC8.2, X7-6.S
- new net S4_RX_33V: D7.C1, IC18.A, R19.1
- net +12V: now also C15.1, C22.1, C29.1, C36.1, C38.1, IC12.VI1, IC16.VI1, IC20.VIN, IC4.V+, IC4.V1+, IC8.VI1, R10.2, R11.2, R8.2, R9.2
- net +3V3: now also C20.1, C27.1, C34.1, C37.1, C39.1, IC10.VCC, IC11P.VCC, IC14.VCC, IC15P.VCC, IC18.VCC, IC19P.VCC, IC20.FB, IC6.VCC, IC7P.VCC, L4.2
- net BATT+: now also IC23.BAT, R20.2, R21.1, R22.2
- net CHARGE: now also C40.1, IC23.!SHDN, IC23.VIN, IC23.VREG
- net GND: now also C15.2, C18.2, C19.1, C20.2, C21.2, C22.2, C25.2, C26.1, C27.2, C28.2, C29.2, C32.2, C33.1, C34.2, C35.2, C36.2, C37.2, C38.2, C39.2, C40.2, C41.2, D10.A, D3.A, D4.A, D5.A, D6.A, D7.A, D8.A, IC10.GND, IC11P.GND, IC12.GND, IC13.GND, IC14.GND, IC15P.GND, IC16.GND, IC17.GND, IC18.GND, IC19P.GND, IC20.GND3, IC20.SD, IC23.GND, IC4.GND, IC4.GND1, IC5.GND, IC6.GND, IC7P.GND, IC8.GND, IC9.GND, R24.1
- net GPIO2A: now also D4.C1, PTC3.1
- net GPIO2B: now also D4.C2, PTC4.1
- net GPIO3A: now also D6.C1, PTC5.1
- net GPIO3B: now also D6.C2, PTC6.1
- net GPIO4A: now also D8.C1, PTC7.1
- net GPIO4B: now also D8.C2, PTC8.1
- net RX1_TTL: now also IC6.Y
- net RX2_TTL: now also IC10.Y, IC7G$1.R1OUT
- net RX3_TTL: now also IC11G$1.R1OUT, IC14.Y
- net RX4_TTL: now also IC15G$1.R1OUT, IC18.Y
- net S1_12V: now also T2.S
- net S1_5V: now also IC5.VCC
- net S1_RX: now also R16.2
- net S1_TX: now also IC5.Y
- net S2_12V: now also T3.S
- net S2_5V: now also C21.1, IC8.VO, IC9.VCC
- net S2_RX: now also IC7G$1.R1IN, R17.2
- net S2_TX: now also IC7G$1.T1OUT, IC9.Y
- net S3_12V: now also T4.S
- net S3_5V: now also C28.1, IC12.VO, IC13.VCC
- net S3_RX: now also IC11G$1.R1IN, R18.2
- net S3_TX: now also IC11G$1.T1OUT, IC13.Y
- net S4_12V: now also T5.S
- net S4_5V: now also C35.1, IC16.VO, IC17.VCC
- net S4_RX: now also IC15G$1.R1IN, R19.2
- net S4_TX: now also IC15G$1.T1OUT, IC17.Y
- net TX1_TTL: now also IC5.A
- net TX2_TTL: now also IC7G$1.T1IN, IC9.A
- net TX3_TTL: now also IC11G$1.T1IN, IC13.A
- net TX4_TTL: now also IC15G$1.T1IN, IC17.A
- net V+: now also R21.2
Other:
- note added: "Replace LT1161 cap"
- note added: "Replace caps and diode (1A rated, 1N5819)"
- note removed: "Add BLMC connections."
- note removed: "Add charging circuit"
- note removed: "Add main power regulator"
- note removed: "Use the: 1.5A PTC on +12V (R1812)"
- note removed: "Use the: LT1161 for +12V"
- note removed: "Use the: SN74LVC1T45?"
- moved on the sheet: C1, C10, C11, C12, C13, C14, C2, C3, C4, C5, C6, C7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

Commit message: Added fixes for current monitoring
Parts:
- added C43, C44: 0.1uF, rcl:C-USC0805
- added C45, C46: 10pF, rcl:C-USC0805
- added R25: 1k, rcl:R-US_R0805
- added R26: 2k, rcl:R-US_R0805
- added R27: 10k, rcl:R-US_R0805
- added X15, X16: 22-23-2021, con-molex:22-23-2021
- R20: value 0.05 -> 0.050
- R21: value 0.05 -> 0.010
- R23: value 0R -> 4.99k
Connections:
- removed net N$43: D9.A, IC23.SENSE, L5.2, R20.1
- removed net N$45: R22.1, R23.1, R24.2
- new net BATT_CURR_IN: C45.1, IC21.OUT, IC3.PA0, R25.2
- new net BATT_CURR_OUT: C46.1, IC22.OUT, IC3.PA1, R23.2
- new net CHRG+: D9.A, IC21.VIN+, IC23.SENSE, L5.2, R20.1
- new net N$48: IC21.R_OS, R26.2
- new net N$49: IC22.R_OS, R27.2
- net +3V3: now also C43.1, C44.1, IC21.V+, IC21.VREF, IC22.V+, IC22.VREF
- net BATT+: now also IC21.VIN-, IC22.VIN+, X15-1.S, X16-1.S
- net BATT-: now also X15-2.S, X16-2.S
- net GND: now also C43.2, C44.2, C45.2, C46.2, IC21.GND, IC22.GND, R23.1, R25.1, R26.1, R27.1
- net N$44: now also R22.1, R24.2; no longer R23.2
- net V+: now also IC22.VIN-
Other:
- note added: "Add battery thermistors"
- note added: "Battery Input Monitor"
- note added: "Battery Output Monitor"
- note added: "TODO: Replace with Deans"
- moved on the sheet: C1, IC21, IC22, L1, R1, R22, R23, R24

Commit message: Added external GPS unit to schematic.
Parts:
- added C47: 10uF, rcl:C-USC0805
- added LED3: GRN, led:LEDCHIPLED_1206
- added R28: 330, rcl:R-US_R0805
- added U2: D2523T_, SparkFun-RF:D2523T_
- LED1: value (none) -> YEL
- LED2: value (none) -> RED
Connections:
- removed net DEBUG_RXD: IC3.PC2
- removed net DEBUG_TXD: IC3.PC3
- new net GPS_RXD: IC3.PC2, U2.TX
- new net GPS_TXD: IC3.PC3, U2.RX
- new net N$43: LED3.C, U2.LED
- new net N$50: LED3.A, R28.1
- net +3V3: now also C47.1, R28.2, U2.VIN
- net GND: now also C47.2, U2.GND
Changed lines of the file:
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@@
 <part name="R2" library="rcl" deviceset="R-US_" device="R0805" value="10k"/>
 <part name="+3V4" library="supply1" deviceset="+3V3" device=""/>
-<part name="LED1" library="led" deviceset="LED" device="CHIPLED_1206"/>
+<part name="LED1" library="led" deviceset="LED" device="CHIPLED_1206" value="YEL"/>
 <part name="R3" library="rcl" deviceset="R-US_" device="R0805" value="330"/>
 <part name="+3V5" library="supply1" deviceset="+3V3" device=""/>
@@
 <part name="+3V6" library="supply1" deviceset="+3V3" device=""/>
 <part name="SUPPLY11" library="supply2" deviceset="GND" device=""/>
-<part name="LED2" library="led" deviceset="LED" device="CHIPLED_1206"/>
+<part name="LED2" library="led" deviceset="LED" device="CHIPLED_1206" value="RED"/>
 <part name="R7" library="rcl" deviceset="R-US_" device="R0805" value="330"/>
 <part name="+3V7" library="supply1" deviceset="+3V3" device=""/>
@@
 <part name="+3V19" library="supply1" deviceset="+3V3" device=""/>
 <part name="+3V20" library="supply1" deviceset="+3V3" device=""/>
+<part name="U2" library="SparkFun-RF" deviceset="D2523T" device="_"/>
+<part name="R28" library="rcl" deviceset="R-US_" device="R0805" value="330"/>
+<part name="LED3" library="led" deviceset="LED" device="CHIPLED_1206" value="GRN"/>
+<part name="C47" library="rcl" deviceset="C-US" device="C0805" value="10uF"/>
+<part name="+3V22" library="supply1" deviceset="+3V3" device=""/>
+<part name="SUPPLY46" library="supply2" deviceset="GND" device=""/>
 </parts>
 <sheets>
@@
 <instance part="+3V19" gate="G$1" x="147.32" y="132.08"/>
 <instance part="+3V20" gate="G$1" x="233.68" y="132.08"/>
+<instance part="U2" gate="G$1" x="490.22" y="195.58" rot="R180"/>
+<instance part="R28" gate="G$1" x="518.16" y="203.2"/>
+<instance part="LED3" gate="G$1" x="508" y="203.2" rot="R270"/>
+<instance part="C47" gate="G$1" x="525.78" y="195.58"/>
+<instance part="+3V22" gate="G$1" x="525.78" y="210.82"/>
+<instance part="SUPPLY46" gate="GND" x="525.78" y="185.42"/>
 </instances>
 <busses>
@@
 <wire x1="279.4" y1="142.24" x2="279.4" y2="139.7" width="0.1524" layer="91"/>
 </segment>
+<segment>
+<pinref part="C47" gate="G$1" pin="2"/>
+<pinref part="SUPPLY46" gate="GND" pin="GND"/>
+<wire x1="525.78" y1="187.96" x2="525.78" y2="190.5" width="0.1524" layer="91"/>
+<pinref part="U2" gate="G$1" pin="GND"/>
+<wire x1="500.38" y1="193.04" x2="520.7" y2="193.04" width="0.1524" layer="91"/>
+<wire x1="520.7" y1="193.04" x2="520.7" y2="190.5" width="0.1524" layer="91"/>
+<wire x1="520.7" y1="190.5" x2="525.78" y2="190.5" width="0.1524" layer="91"/>
+<junction x="525.78" y="190.5"/>
+</segment>
 </net>
 <net name="S1_12V" class="0">
@@
 <wire x1="233.68" y1="129.54" x2="238.76" y2="129.54" width="0.1524" layer="91"/>
 </segment>
+<segment>
+<pinref part="C47" gate="G$1" pin="1"/>
+<pinref part="+3V22" gate="G$1" pin="+3V3"/>
+<wire x1="525.78" y1="208.28" x2="525.78" y2="203.2" width="0.1524" layer="91"/>
+<pinref part="R28" gate="G$1" pin="2"/>
+<wire x1="525.78" y1="203.2" x2="525.78" y2="198.12" width="0.1524" layer="91"/>
+<wire x1="523.24" y1="203.2" x2="525.78" y2="203.2" width="0.1524" layer="91"/>
+<junction x="525.78" y="203.2"/>
+<pinref part="U2" gate="G$1" pin="VIN"/>
+<wire x1="500.38" y1="195.58" x2="520.7" y2="195.58" width="0.1524" layer="91"/>
+<wire x1="520.7" y1="195.58" x2="520.7" y2="198.12" width="0.1524" layer="91"/>
+<wire x1="520.7" y1="198.12" x2="525.78" y2="198.12" width="0.1524" layer="91"/>
+<junction x="525.78" y="198.12"/>
+</segment>
 </net>
 <net name="+12V" class="0">
@@
 </segment>
 </net>
-<net name="DEBUG_RXD" class="0">
+<net name="GPS_RXD" class="0">
 <segment>
 <pinref part="IC3" gate="G$1" pin="PC2"/>
@@
 <label x="114.3" y="347.98" size="1.778" layer="95"/>
 </segment>
+<segment>
+<pinref part="U2" gate="G$1" pin="TX"/>
+<wire x1="500.38" y1="190.5" x2="515.62" y2="190.5" width="0.1524" layer="91"/>
+<label x="502.92" y="190.5" size="1.778" layer="95"/>
+</segment>
 </net>
-<net name="DEBUG_TXD" class="0">
+<net name="GPS_TXD" class="0">
 <segment>
 <pinref part="IC3" gate="G$1" pin="PC3"/>
@@
 <label x="114.3" y="350.52" size="1.778" layer="95"/>
 </segment>
+<segment>
+<pinref part="U2" gate="G$1" pin="RX"/>
+<wire x1="500.38" y1="187.96" x2="515.62" y2="187.96" width="0.1524" layer="91"/>
+<label x="502.92" y="187.96" size="1.778" layer="95"/>
+</segment>
 </net>
 <net name="BT_RXD" class="0">
@@
 </segment>
 </net>
+<net name="N$50" class="0">
+<segment>
+<pinref part="LED3" gate="G$1" pin="A"/>
+<pinref part="R28" gate="G$1" pin="1"/>
+<wire x1="513.08" y1="203.2" x2="510.54" y2="203.2" width="0.1524" layer="91"/>
+</segment>
+</net>
+<net name="N$43" class="0">
+<segment>
+<pinref part="LED3" gate="G$1" pin="C"/>
+<pinref part="U2" gate="G$1" pin="LED"/>
+<wire x1="502.92" y1="203.2" x2="500.38" y2="203.2" width="0.1524" layer="91"/>
+<wire x1="500.38" y1="203.2" x2="500.38" y2="200.66" width="0.1524" layer="91"/>
+</segment>
+</net>

Commit message: Added missing batt_temp connector.
Parts:
- added X17: 22-23-2021, con-molex:22-23-2021
Connections:
- net BATT_TEMP: now also IC3.PA2, X17-1.S
- net GND: now also X17-2.S
Other:
- moved on the sheet: C47, LED3, R28, U2
Changed lines of the file:
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@@
 <part name="+3V22" library="supply1" deviceset="+3V3" device=""/>
 <part name="SUPPLY46" library="supply2" deviceset="GND" device=""/>
+<part name="X17" library="con-molex" deviceset="22-23-2021" device=""/>
+<part name="SUPPLY47" library="supply2" deviceset="GND" device=""/>
 </parts>
 <sheets>
@@
 <instance part="+3V19" gate="G$1" x="147.32" y="132.08"/>
 <instance part="+3V20" gate="G$1" x="233.68" y="132.08"/>
-<instance part="U2" gate="G$1" x="490.22" y="195.58" rot="R180"/>
-<instance part="R28" gate="G$1" x="518.16" y="203.2"/>
-<instance part="LED3" gate="G$1" x="508" y="203.2" rot="R270"/>
-<instance part="C47" gate="G$1" x="525.78" y="195.58"/>
-<instance part="+3V22" gate="G$1" x="525.78" y="210.82"/>
-<instance part="SUPPLY46" gate="GND" x="525.78" y="185.42"/>
+<instance part="U2" gate="G$1" x="490.22" y="180.34" rot="R180"/>
+<instance part="R28" gate="G$1" x="518.16" y="187.96"/>
+<instance part="LED3" gate="G$1" x="508" y="187.96" rot="R270"/>
+<instance part="C47" gate="G$1" x="525.78" y="180.34"/>
+<instance part="+3V22" gate="G$1" x="525.78" y="195.58"/>
+<instance part="SUPPLY46" gate="GND" x="525.78" y="170.18"/>
+<instance part="X17" gate="-1" x="497.84" y="208.28" rot="MR0"/>
+<instance part="X17" gate="-2" x="497.84" y="205.74" rot="MR0"/>
+<instance part="SUPPLY47" gate="GND" x="515.62" y="203.2"/>
 </instances>
 <busses>
@@
 <pinref part="C47" gate="G$1" pin="2"/>
 <pinref part="SUPPLY46" gate="GND" pin="GND"/>
-<wire x1="525.78" y1="187.96" x2="525.78" y2="190.5" width="0.1524" layer="91"/>
+<wire x1="525.78" y1="172.72" x2="525.78" y2="175.26" width="0.1524" layer="91"/>
 <pinref part="U2" gate="G$1" pin="GND"/>
-<wire x1="500.38" y1="193.04" x2="520.7" y2="193.04" width="0.1524" layer="91"/>
-<wire x1="520.7" y1="193.04" x2="520.7" y2="190.5" width="0.1524" layer="91"/>
-<wire x1="520.7" y1="190.5" x2="525.78" y2="190.5" width="0.1524" layer="91"/>
-<junction x="525.78" y="190.5"/>
+<wire x1="500.38" y1="177.8" x2="520.7" y2="177.8" width="0.1524" layer="91"/>
+<wire x1="520.7" y1="177.8" x2="520.7" y2="175.26" width="0.1524" layer="91"/>
+<wire x1="520.7" y1="175.26" x2="525.78" y2="175.26" width="0.1524" layer="91"/>
+<junction x="525.78" y="175.26"/>
+</segment>
+<segment>
+<pinref part="X17" gate="-2" pin="S"/>
+<wire x1="500.38" y1="205.74" x2="515.62" y2="205.74" width="0.1524" layer="91"/>
+<pinref part="SUPPLY47" gate="GND" pin="GND"/>
 </segment>
 </net>
@@
 <pinref part="C47" gate="G$1" pin="1"/>
 <pinref part="+3V22" gate="G$1" pin="+3V3"/>
-<wire x1="525.78" y1="208.28" x2="525.78" y2="203.2" width="0.1524" layer="91"/>
+<wire x1="525.78" y1="193.04" x2="525.78" y2="187.96" width="0.1524" layer="91"/>
 <pinref part="R28" gate="G$1" pin="2"/>
-<wire x1="525.78" y1="203.2" x2="525.78" y2="198.12" width="0.1524" layer="91"/>
-<wire x1="523.24" y1="203.2" x2="525.78" y2="203.2" width="0.1524" layer="91"/>
-<junction x="525.78" y="203.2"/>
+<wire x1="525.78" y1="187.96" x2="525.78" y2="182.88" width="0.1524" layer="91"/>
+<wire x1="523.24" y1="187.96" x2="525.78" y2="187.96" width="0.1524" layer="91"/>
+<junction x="525.78" y="187.96"/>
 <pinref part="U2" gate="G$1" pin="VIN"/>
-<wire x1="500.38" y1="195.58" x2="520.7" y2="195.58" width="0.1524" layer="91"/>
-<wire x1="520.7" y1="195.58" x2="520.7" y2="198.12" width="0.1524" layer="91"/>
-<wire x1="520.7" y1="198.12" x2="525.78" y2="198.12" width="0.1524" layer="91"/>
-<junction x="525.78" y="198.12"/>
+<wire x1="500.38" y1="180.34" x2="520.7" y2="180.34" width="0.1524" layer="91"/>
+<wire x1="520.7" y1="180.34" x2="520.7" y2="182.88" width="0.1524" layer="91"/>
+<wire x1="520.7" y1="182.88" x2="525.78" y2="182.88" width="0.1524" layer="91"/>
+<junction x="525.78" y="182.88"/>
 </segment>
 </net>
@@
 <segment>
 <pinref part="U2" gate="G$1" pin="TX"/>
-<wire x1="500.38" y1="190.5" x2="515.62" y2="190.5" width="0.1524" layer="91"/>
-<label x="502.92" y="190.5" size="1.778" layer="95"/>
+<wire x1="500.38" y1="175.26" x2="515.62" y2="175.26" width="0.1524" layer="91"/>
+<label x="502.92" y="175.26" size="1.778" layer="95"/>
 </segment>
 </net>
@@
 <segment>
 <pinref part="U2" gate="G$1" pin="RX"/>
-<wire x1="500.38" y1="187.96" x2="515.62" y2="187.96" width="0.1524" layer="91"/>
-<label x="502.92" y="187.96" size="1.778" layer="95"/>
+<wire x1="500.38" y1="172.72" x2="515.62" y2="172.72" width="0.1524" layer="91"/>
+<label x="502.92" y="172.72" size="1.778" layer="95"/>
 </segment>
 </net>
@@
 <label x="190.5" y="58.42" size="1.778" layer="95"/>
 </segment>
+<segment>
+<pinref part="X17" gate="-1" pin="S"/>
+<wire x1="500.38" y1="208.28" x2="518.16" y2="208.28" width="0.1524" layer="91"/>
+<label x="502.92" y="208.28" size="1.778" layer="95"/>
+</segment>
+<segment>
+<pinref part="IC3" gate="G$1" pin="PA2"/>
+<wire x1="111.76" y1="393.7" x2="137.16" y2="393.7" width="0.1524" layer="91"/>
+<label x="114.3" y="393.7" size="1.778" layer="95"/>
+</segment>
 </net>
 <net name="BATT_CURR_IN" class="0">
@@
 <pinref part="LED3" gate="G$1" pin="A"/>
 <pinref part="R28" gate="G$1" pin="1"/>
-<wire x1="513.08" y1="203.2" x2="510.54" y2="203.2" width="0.1524" layer="91"/>
+<wire x1="513.08" y1="187.96" x2="510.54" y2="187.96" width="0.1524" layer="91"/>
 </segment>
 </net>
@@
 <pinref part="LED3" gate="G$1" pin="C"/>
 <pinref part="U2" gate="G$1" pin="LED"/>
-<wire x1="502.92" y1="203.2" x2="500.38" y2="203.2" width="0.1524" layer="91"/>
-<wire x1="500.38" y1="203.2" x2="500.38" y2="200.66" width="0.1524" layer="91"/>
-</segment>
-</net>
+<wire x1="502.92" y1="187.96" x2="500.38" y2="187.96" width="0.1524" layer="91"/>
+<wire x1="500.38" y1="187.96" x2="500.38" y2="185.42" width="0.1524" layer="91"/>
+</segment>
+</net>
