File: electrical/ebox/ebox.sch (EAGLE design)
At the start: 152 parts, among them IC1 MAX3221CUE, IC10 SN74LVC1G125, IC11 MAX3221CUE, IC12 MCP170350MB, IC13 SN74LVC1G125, IC14 SN74LVC1G125, IC15 MAX3221CUE, IC16 MCP170350MB, IC17 SN74LVC1G125, IC18 SN74LVC1G125, IC19 74ALS04D, IC2 MCP170350MB, IC20 AP1509-33, IC23 LT3652, IC3 XMEGA128A1, IC4 LT1161, IC5 SN74LVC1G125, IC6 SN74LVC1G125, IC7 MAX3221CUE, IC8 MCP170350MB, IC9 SN74LVC1G125, Q1 FDD4141TO252, U1 BLUETOOTH-RN42, U2 D2523T_, X1 22-23-2031, X10 22-23-2041, X11 22-23-2041, X12 22-23-2021, X13 22-23-2031, X14 22-23-2031, X15 22-23-2021, X16 22-23-2021, X17 22-23-2021, X2 22-23-2031, X3 C-GRID-07-70543, X4 22-23-2031, X5 C-GRID-07-70543, X6 C-GRID-07-70543, X7 C-GRID-07-70543, X8 22-23-2031, X9 22-23-2031

Commit message: Fixed most footprints.  Still have to do a couple of connectors, then should be good to go.
Parts:
- removed C1: (no value), rcl:C-USC0805
- removed C35, C36: 1uF, rcl:C-USC0805
- removed C38: 68uF, rcl:C-USC0805
- removed C39: 120uF, rcl:C-USC0805
- removed C40: 10uF, rcl:C-USC0805
- removed IC12, IC16, IC2, IC8: MCP170350MB, linear:MCP170350MB
- removed L1: (no value), rcl:L-USL2012C
- removed X10, X11: 22-23-2041, con-molex:22-23-2041
- added C48: 10pF, rcl:C-USC0805
- added D11, D12: MBRA340T3, diode:MBRA340T3
- added IC24: AP1509-5, crw:AP1509
- added L6: 47uH, rcl:L-USL2012C
- added LED4: RED, led:LEDCHIPLED_1206
- added LED6: (no value), led:TOPLED-3P-LCC-4
- added PTC10, PTC11, PTC12, PTC9: 1A, rcl:R-US_R1206
- added R29: 10k, rcl:R-US_R0805
- added R30: 2k, rcl:R-US_R0805
- added R31, R32, R33: 330, rcl:R-US_R0805
- added X18, X19: 7381-3PG-300, crw:7381-3PG-300
- added X20, X21, X22, X23: BULLET, crw:BULLET
- added X24: B4B-ZR, con-jst:B4B-ZR
- C15: value 50uF -> 68uF; device rcl:C-USC0805 -> rcl:CPOL-USD
- C21, C29, C8: value 1uF -> 68uF; device rcl:C-USC0805 -> rcl:CPOL-USD
- C22, C28: value 1uF -> 220uF; device rcl:C-USC0805 -> rcl:CPOL-USD
- R1: value (none) -> 330
- X1, X14, X2, X4: value 22-23-2031 -> BULLET; device con-molex:22-23-2031 -> crw:BULLET
- X12: value 22-23-2021 -> 7381-3PG-300; device con-molex:22-23-2021 -> crw:7381-3PG-300
- X13: value 22-23-2031 -> B4B-ZR; device con-molex:22-23-2031 -> con-jst:B4B-ZR
Connections:
- removed net MOT_SERVO1: IC3.PF0
- removed net MOT_SERVO2: IC3.PF1
- new net +5V: C28.+, IC24.FB, L6.2, PTC10.1, PTC11.1, PTC12.1, PTC9.1
- new net BATT_VSENSE: C48.1, IC3.PA3, R29.1, R30.2
- new net BT_CTS: IC3.PF4, U1.UARTCTS
- new net BT_RTS: IC3.PF5, U1.UARTRTS
- new net N$45: D11.C, IC24.OUT, L6.1
- new net N$46: LED4.A, R1.1
- new net N$47: C29.+, C7.1, D12.C, IC23.!SHDN, IC23.VIN, IC23.VREG
- new net N$51: LED6.CBLUE, R32.2
- new net N$52: LED6.CRED, R31.2
- new net N$53: LED6.CGREEN, R33.2
- net +12V: now also C15.+, C21.+, C8.+, IC24.VIN; no longer C15.1, C22.1, C29.1, C36.1, C38.1, C7.1, IC12.VI1, IC16.VI1, IC2.VI1, IC8.VI1
- net +3V3: now also C22.+, LED6.A2, R1.2; no longer C39.1
- net BATT+: now also R29.2, X13-4.1, X24-4.1; no longer X10-1.S, X11-1.S
- net BATT-: now also X13-1.1, X24-1.1; no longer X10-4.S, X11-4.S
- net BATT1: now also X13-2.1, X24-2.1; no longer X10-3.S, X11-3.S
- net BATT2: now also X13-3.1, X24-3.1; no longer X10-2.S, X11-2.S
- net BT_RESET: now also IC3.PF6; no longer IC3.PJ0
- net BT_STATUS: now also IC3.PF7; no longer IC3.PJ1
- net CHARGE: now also D12.A, X4.S; no longer C40.1, IC23.!SHDN, IC23.VIN, IC23.VREG, X13-1.S
- net GND: now also C15.-, C21.-, C22.-, C28.-, C29.-, C48.2, C8.-, D11.A, IC19E.I, IC19F.I, IC20.GND, IC20.GND1, IC20.GND2, IC24.GND, IC24.GND1, IC24.GND2, IC24.GND3, IC24.SD, LED4.C, R30.1, X14.S; no longer C15.2, C21.2, C22.2, C28.2, C29.2, C35.2, C36.2, C38.2, C39.2, C40.2, C8.2, IC12.GND, IC16.GND, IC2.GND, IC8.GND, X13-2.S
- net LED_BLU: now also R32.1
- net LED_GRN: now also R33.1
- net LED_RED: now also R31.1
- net MOT1_A: now also X1.S, X18-1.S; no longer X1-1.S, X4-1.S
- net MOT1_B: now also X18-2.S, X2.S; no longer X1-2.S, X4-2.S
- net MOT1_C: now also X18-3.S, X20.S; no longer X1-3.S, X4-3.S
- net MOT1_SIG: now also IC3.PF0
- net MOT2_A: now also X19-1.S, X21.S; no longer X14-1.S, X2-1.S
- net MOT2_B: now also X19-2.S, X22.S; no longer X14-2.S, X2-2.S
- net MOT2_C: now also X19-3.S, X23.S; no longer X14-3.S, X2-3.S
- net MOT2_SIG: now also IC3.PF1
- net N$12: now also IC4.DS1
- net N$14: now also IC4.DS2
- net N$15: now also IC4.DS3
- net N$16: now also IC4.DS4
- net S1_5V: now also PTC9.2; no longer C8.1, IC2.VO
- net S2_5V: now also PTC10.2; no longer C21.1, IC8.VO
- net S3_5V: now also PTC11.2; no longer C28.1, IC12.VO
- net S4_5V: now also PTC12.2; no longer C35.1, IC16.VO
Other:
- note added: "TODO: Check hole size on mini-con-X"
- note added: "TODO: Replace charge w/ 2-pin mini-con-X"
- note added: "TODO: Replace with micro-con-X"
- note removed: "Add battery thermistors"
- note removed: "Replace LT1161 cap"
- note removed: "TODO: Replace with JST"
- note removed: "TODO: Replace with bullet"
- note removed: "TODO: Replace with mini-con-x"
- note removed: "TODO: Replace with multi-con-X"
- note removed: "Use Mike's LED Strips?"
- moved on the sheet: C37, C41, C42, C7, D10, D3, D7, D9, IC19A, IC19B, IC19C, IC19D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

Commit message: Added all footprints (still need to fix micro-con) and repaired most ERC errors.
Parts:
- removed X15, X16: 22-23-2021, con-molex:22-23-2021
- added X10, X11: DEANS, crw:DEANS
- IC12, IC8: value (none) -> INA170
- X12: value 7381-3PG-300 -> 7381-2PG-300; device crw:7381-3PG-300 -> crw:7381-2PG-300
- X3, X5, X6, X7: value C-GRID-07-70543 -> 17984-7PG-300; device con-molex:C-GRID-07-70543 -> crw:17984-7PG-300
- renumbered IC21 to IC8, IC22 to IC12, IC23 to IC2
Connections:
- net BATT+: now also X10-POS.S, X11-POS.S; no longer X15-1.S, X16-1.S
- net BATT-: now also X10-NEG.S, X11-NEG.S; no longer X15-2.S, X16-2.S
Other:
- note added: "TODO: Fix micro-con-X footprint"
- note removed: "Replace caps and diode (1A rated, 1N5819)"
- note removed: "TODO: Check hole size on mini-con-X"
- note removed: "TODO: Replace charge w/ 2-pin mini-con-X"
- note removed: "TODO: Replace with Deans"
- note removed: "TODO: Replace with micro-con-X"

Commit message: Added board and some of layout.
Parts:
- removed L4, L6: 47uH, rcl:L-USL2012C
- added L1: 5.6uH, crw:IHLP-2020CZ-11
- added L7: 47uH, crw:L-SRR1280
- L5: value 5.6uH -> 47uH; device rcl:L-USL2012C -> crw:L-SRR1280
Connections:
- net +3V3: now also L7.2; no longer L4.2
- net +5V: now also L5.2; no longer L6.2
- net CHRG+: now also L1.2; no longer L5.2
- net N$40: now also L7.1; no longer L4.1
- net N$42: now also L1.1; no longer L5.1
- net N$45: now also L5.1; no longer L6.1
Other:
- moved on the sheet: D10, L5
Changed lines of the file:
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@@
 <part name="IC20" library="crw" deviceset="AP1509" device="" value="AP1509-33"/>
 <part name="P+8" library="supply1" deviceset="+12V" device=""/>
-<part name="L4" library="rcl" deviceset="L-US" device="L2012C" value="47uH"/>
 <part name="D5" library="diode" deviceset="MBRA340T3" device=""/>
 <part name="+3V16" library="supply1" deviceset="+3V3" device=""/>
@@
 <part name="SUPPLY39" library="supply2" deviceset="GND" device=""/>
 <part name="C42" library="rcl" deviceset="C-US" device="C0805" value="1uF"/>
-<part name="L5" library="rcl" deviceset="L-US" device="L2012C" value="5.6uH"/>
 <part name="R20" library="rcl" deviceset="R-US_" device="R6332" value="0.050"/>
 <part name="P+9" library="supply1" deviceset="V+" device=""/>
@@
 <part name="IC24" library="crw" deviceset="AP1509" device="" value="AP1509-5"/>
 <part name="P+10" library="supply1" deviceset="+12V" device=""/>
-<part name="L6" library="rcl" deviceset="L-US" device="L2012C" value="47uH"/>
 <part name="D11" library="diode" deviceset="MBRA340T3" device=""/>
 <part name="SUPPLY49" library="supply2" deviceset="GND" device=""/>
@@
 <part name="IC8" library="crw" deviceset="INA170" device=""/>
 <part name="IC12" library="crw" deviceset="INA170" device=""/>
+<part name="L1" library="crw" deviceset="IHLP-2020CZ-11" device="" value="5.6uH"/>
+<part name="L5" library="crw" deviceset="L" device="-SRR1280" value="47uH"/>
+<part name="L7" library="crw" deviceset="L" device="-SRR1280" value="47uH"/>
 </parts>
 <sheets>
@@
 <instance part="IC20" gate="G$1" x="73.66" y="58.42"/>
 <instance part="P+8" gate="1" x="45.72" y="68.58"/>
-<instance part="L4" gate="G$1" x="99.06" y="60.96" rot="R90"/>
 <instance part="D5" gate="G$1" x="88.9" y="48.26" rot="R90"/>
 <instance part="+3V16" gate="G$1" x="116.84" y="68.58"/>
@@
 <instance part="SUPPLY39" gate="GND" x="266.7" y="30.48"/>
 <instance part="C42" gate="G$1" x="304.8" y="76.2"/>
-<instance part="L5" gate="G$1" x="332.74" y="73.66"/>
 <instance part="R20" gate="G$1" x="342.9" y="63.5"/>
 <instance part="P+9" gate="1" x="365.76" y="71.12"/>
@@
 <instance part="SUPPLY41" gate="GND" x="320.04" y="33.02"/>
 <instance part="D9" gate="G$1" x="322.58" y="68.58" rot="R180"/>
-<instance part="D10" gate="G$1" x="337.82" y="81.28" rot="R180"/>
-<instance part="SUPPLY42" gate="GND" x="342.9" y="73.66"/>
+<instance part="D10" gate="G$1" x="347.98" y="81.28" rot="R180"/>
+<instance part="SUPPLY42" gate="GND" x="353.06" y="73.66"/>
 <instance part="R23" gate="G$1" x="289.56" y="124.46" rot="R90"/>
 <instance part="R25" gate="G$1" x="203.2" y="124.46" rot="R90"/>
@@
 <instance part="IC24" gate="G$1" x="165.1" y="58.42"/>
 <instance part="P+10" gate="1" x="137.16" y="68.58"/>
-<instance part="L6" gate="G$1" x="190.5" y="60.96" rot="R90"/>
 <instance part="D11" gate="G$1" x="180.34" y="48.26" rot="R90"/>
 <instance part="SUPPLY49" gate="GND" x="142.24" y="38.1"/>
@@
 <instance part="IC8" gate="G$1" x="165.1" y="132.08"/>
 <instance part="IC12" gate="G$1" x="251.46" y="132.08"/>
+<instance part="L1" gate="G$1" x="332.74" y="73.66"/>
+<instance part="L5" gate="G$1" x="190.5" y="60.96" rot="R90"/>
+<instance part="L7" gate="G$1" x="99.06" y="60.96" rot="R90"/>
 </instances>
 <busses>
@@
 <segment>
 <pinref part="D10" gate="G$1" pin="A"/>
-<wire x1="340.36" y1="81.28" x2="342.9" y2="81.28" width="0.1524" layer="91"/>
-<wire x1="342.9" y1="81.28" x2="342.9" y2="76.2" width="0.1524" layer="91"/>
+<wire x1="350.52" y1="81.28" x2="353.06" y2="81.28" width="0.1524" layer="91"/>
+<wire x1="353.06" y1="81.28" x2="353.06" y2="76.2" width="0.1524" layer="91"/>
 <pinref part="SUPPLY42" gate="GND" pin="GND"/>
 </segment>
@@
 </segment>
 <segment>
-<pinref part="L4" gate="G$1" pin="2"/>
 <wire x1="106.68" y1="60.96" x2="109.22" y2="60.96" width="0.1524" layer="91"/>
 <wire x1="109.22" y1="60.96" x2="116.84" y2="60.96" width="0.1524" layer="91"/>
@@
 <wire x1="116.84" y1="60.96" x2="121.92" y2="60.96" width="0.1524" layer="91"/>
 <junction x="116.84" y="60.96"/>
+<pinref part="L7" gate="G$1" pin="2"/>
 </segment>
 <segment>
@@
 <wire x1="86.36" y1="60.96" x2="88.9" y2="60.96" width="0.1524" layer="91"/>
 <wire x1="88.9" y1="60.96" x2="88.9" y2="50.8" width="0.1524" layer="91"/>
-<pinref part="L4" gate="G$1" pin="1"/>
 <wire x1="88.9" y1="60.96" x2="91.44" y2="60.96" width="0.1524" layer="91"/>
 <junction x="88.9" y="60.96"/>
+<pinref part="L7" gate="G$1" pin="1"/>
 </segment>
 </net>
@@
 <wire x1="299.72" y1="81.28" x2="304.8" y2="81.28" width="0.1524" layer="91"/>
 <wire x1="304.8" y1="81.28" x2="332.74" y2="81.28" width="0.1524" layer="91"/>
+<wire x1="332.74" y1="81.28" x2="345.44" y2="81.28" width="0.1524" layer="91"/>
 <wire x1="297.18" y1="73.66" x2="299.72" y2="73.66" width="0.1524" layer="91"/>
 <wire x1="299.72" y1="81.28" x2="299.72" y2="73.66" width="0.1524" layer="91"/>
-<pinref part="L5" gate="G$1" pin="1"/>
 <pinref part="C42" gate="G$1" pin="1"/>
 <wire x1="304.8" y1="78.74" x2="304.8" y2="81.28" width="0.1524" layer="91"/>
 <junction x="304.8" y="81.28"/>
 <pinref part="D10" gate="G$1" pin="C"/>
-<wire x1="332.74" y1="81.28" x2="335.28" y2="81.28" width="0.1524" layer="91"/>
-<junction x="332.74" y="81.28"/>
 <pinref part="IC2" gate="G$1" pin="SW"/>
+<pinref part="L1" gate="G$1" pin="1"/>
+<junction x="332.74" y="81.28"/>
 </segment>
 </net>
@@
 <segment>
 <wire x1="297.18" y1="63.5" x2="327.66" y2="63.5" width="0.1524" layer="91"/>
-<pinref part="L5" gate="G$1" pin="2"/>
 <wire x1="327.66" y1="63.5" x2="332.74" y2="63.5" width="0.1524" layer="91"/>
 <wire x1="332.74" y1="63.5" x2="332.74" y2="66.04" width="0.1524" layer="91"/>
@@
 <label x="299.72" y="63.5" size="1.778" layer="95"/>
 <pinref part="IC2" gate="G$1" pin="SENSE"/>
+<pinref part="L1" gate="G$1" pin="2"/>
 </segment>
 <segment>
@@
 <wire x1="177.8" y1="60.96" x2="180.34" y2="60.96" width="0.1524" layer="91"/>
 <wire x1="180.34" y1="60.96" x2="180.34" y2="50.8" width="0.1524" layer="91"/>
-<pinref part="L6" gate="G$1" pin="1"/>
 <wire x1="180.34" y1="60.96" x2="182.88" y2="60.96" width="0.1524" layer="91"/>
 <junction x="180.34" y="60.96"/>
+<pinref part="L5" gate="G$1" pin="1"/>
 </segment>
 </net>
 <net name="+5V" class="0">
 <segment>
-<pinref part="L6" gate="G$1" pin="2"/>
 <wire x1="198.12" y1="60.96" x2="200.66" y2="60.96" width="0.1524" layer="91"/>
 <wire x1="200.66" y1="60.96" x2="208.28" y2="60.96" width="0.1524" layer="91"/>
@@
 <pinref part="P+1" gate="1" pin="+5V"/>
 <pinref part="C28" gate="G$1" pin="+"/>
+<pinref part="L5" gate="G$1" pin="2"/>
 </segment>
 <segment>
